File: pico-2v.kicad_pcb (KiCad board)
At the start: 4 copper layers, 51.5 x 21 mm, 50 parts, among them J1 USB_C_Receptacle_USB2.0_16P, J2 VOLTSEL, J3 Header-1, J4 Header-2, J5 Conn_01x04, J6 Conn_01x04, J7 Conn_02x05_Odd_Even, SW1 UK-B0273-SP25Y, SW2 USB Boot, U1 RP2354A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

Commit message: Stuff
Parts:
- added D2: RED, LED_SMD:LED_0603_1608Metric, F.Cu at (135.4, 92.1)
- added R12: 470R, Resistor_SMD:R_0402_1005Metric, F.Cu at (132.9, 92.1)
- added REF**: FireEmoji, pico-2v:FireEmoji, B.Cu at (127.9, 99.2)
- moved R1 2.50 mm to (144.2, 105.5)
- moved R2 2.50 mm to (146.2, 105.5)
- moved SW2 1.80 mm to (150.8, 104.0)
- moved SW1 1.75 mm to (150.8, 93.8)
- moved C5 0.90 mm to (155.5, 95.5), turned to 180 degrees
- turned R3 to 90 degrees
- turned R4 to -90 degrees
Connections:
- R3 pad 1: USB_D+ -> /USB_DP
- R4 pad 2: USB_D- -> /USB_DM
- U1 pad 37: unconnected-(U1-GPIO25-Pad37) -> GPIO25
- U1 pad 51: USB_D- -> /USB_DM
- U1 pad 52: USB_D+ -> /USB_DP
Routing:
- net +3V3: track 14.8 -> 97.6 mm, vias 0 -> 7
- net +1V1: track 7.01 -> 65.5 mm, vias 0 -> 3
- net GPIO25: track 0.00 -> 38.2 mm, vias 0 -> 2
- net +1V8: track 1.47 -> 29.0 mm, vias 0 -> 3
- net SWDIO: track 4.48 -> 29.1 mm, vias 1 -> 2
- net RUN: track 19.6 -> 44.1 mm, vias 3 -> 1
- net QSPI_SD3: track 0.00 -> 23.9 mm, vias 0 -> 1
- net QSPI_SD2: track 0.00 -> 19.8 mm, vias 0 -> 1
- net QSPI_SCLK: track 0.00 -> 19.7 mm, vias 0 -> 1
- net GPIO16: track 51.4 -> 32.6 mm, vias 3 -> 1
- net QSPI_SD1: track 8.11 -> 21.8 mm
- net VDD: track 27.7 -> 39.8 mm, vias 5 -> 10
- net GPIO18: track 14.4 -> 23.7 mm
- net QSPI_SD0: track 7.73 -> 16.5 mm
- net GPIO19: track 17.2 -> 22.2 mm
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Other:
- board text added: "LED"
- board text added: "Pico 2V by Lucas Baizer"
- board text added: "QSPI"
- board text added: "rev. 0"

Commit message: Bug fixes
Routing:
- net GPIO21: track 18.8 -> 17.2 mm
Changed lines of the file:
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@@
 	)
 	(segment
-		(start 164.629904 104.669904)
-		(end 165.21 105.25)
+		(start 141.75 101)
+		(end 148.5 101)
 		(width 0.3)
 		(layer "B.Cu")
@@
 	)
 	(segment
-		(start 149.73343 104.669904)
+		(start 151.890672 104.669904)
 		(end 164.629904 104.669904)
 		(width 0.3)
@@
 	)
 	(segment
-		(start 172 102.8)
-		(end 171.85 102.65)
+		(start 164.629904 104.669904)
+		(end 165.21 105.25)
 		(width 0.3)
 		(layer "B.Cu")
@@
 	)
 	(segment
-		(start 171.85 102.65)
-		(end 168.8 102.65)
+		(start 149 101.779232)
+		(end 151.890672 104.669904)
+		(width 0.3)
+		(layer "B.Cu")
+		(net 1)
+	)
+	(segment
+		(start 172 102.8)
+		(end 171.85 102.65)
 		(width 0.3)
 		(layer "B.Cu")
@@
 	)
 	(segment
-		(start 149.704334 104.699)
-		(end 146.005334 101)
+		(start 171.85 102.65)
+		(end 168.8 102.65)
 		(width 0.3)
 		(layer "B.Cu")
@@
 	)
 	(segment
-		(start 146.005334 101)
-		(end 141.75 101)
+		(start 148.5 101)
+		(end 149 101.5)
 		(width 0.3)
 		(layer "B.Cu")
@@
 	)
 	(segment
-		(start 149.704334 104.699)
-		(end 149.73343 104.669904)
+		(start 149 101.5)
+		(end 149 101.779232)
 		(width 0.3)
 		(layer "B.Cu")
@@
 	)
 	(via
-		(at 149.75 101.75)
-		(size 0.45)
-		(drill 0.3)
-		(layers "F.Cu" "B.Cu")
-		(free yes)
-		(net 2)
-	)
-	(via
 		(at 166.25 93.5)
 		(size 0.45)
@@
 	)
 	(via
+		(at 148.7 103.25)
+		(size 0.45)
+		(drill 0.3)
+		(layers "F.Cu" "B.Cu")
+		(net 2)
+	)
+	(via
 		(at 155.02 95.5)
 		(size 0.45)
@@
 	)
 	(segment
+		(start 149.25 99.46296)
+		(end 149.25 100.5)
+		(width 0.3)
+		(layer "B.Cu")
+		(net 6)
+	)
+	(segment
 		(start 169.169 104.129)
 		(end 152.879 104.129)
@@
 	)
 	(segment
-		(start 149.25 99.46296)
-		(end 149.25 100.5)
-		(width 0.3)
-		(layer "In2.Cu")
-		(net 6)
-	)
-	(segment
 		(start 155.71 92)
 		(end 155.71 92.72)
@@
 	)
 	(segment
-		(start 149.904616 103.75)
-		(end 150.592232 103.062384)
+		(start 136.044334 103.801)
+		(end 135.993334 103.75)
 		(width 0.3)
 		(layer "In1.Cu")
@@
 	)
 	(segment
-		(start 135.993334 103.75)
-		(end 149.904616 103.75)
+		(start 149.853616 103.801)
+		(end 136.044334 103.801)
 		(width 0.3)
 		(layer "In1.Cu")
@@
 	(segment
 		(start 133.084334 106.659)
-		(end 135.993334 103.75)
+		(end 128.661 106.659)
 		(width 0.3)
 		(layer "In1.Cu")
@@
 	)
 	(segment
-		(start 150.592232 103.062384)
-		(end 150.592232 99.907768)
+		(start 128.661 106.659)
+		(end 127.54 107.78)
 		(width 0.3)
 		(layer "In1.Cu")
@@
 	)
 	(segment
-		(start 127.54 107.78)
-		(end 128.661 106.659)
+		(start 150.592232 99.907768)
+		(end 150.592232 103.062384)
 		(width 0.3)
 		(layer "In1.Cu")
@@
 	)
 	(segment
-		(start 128.661 106.659)
-		(end 133.084334 106.659)
+		(start 153 97.5)
+		(end 150.592232 99.907768)
 		(width 0.3)
 		(layer "In1.Cu")
@@
 	)
 	(segment
-		(start 150.592232 99.907768)
-		(end 153 97.5)
+		(start 150.592232 103.062384)
+		(end 149.853616 103.801)
+		(width 0.3)
+		(layer "In1.Cu")
+		(net 24)
+	)
+	(segment
+		(start 135.993334 103.75)
+		(end 133.084334 106.659)
 		(width 0.3)
 		(layer "In1.Cu")
@@
 	)
 	(segment
+		(start 164.9 100.5)
+		(end 165.4 100)
+		(width 0.2)
+		(layer "F.Cu")
+		(net 33)
+	)
+	(segment
 		(start 164.1375 100.5)
-		(end 163.715362 100.5)
+		(end 164.9 100.5)
 		(width 0.2)
 		(layer "F.Cu")
@@
 	)
 	(via
-		(at 163.25 98.5)
+		(at 165.4 100)
 		(size 0.45)
 		(drill 0.3)
@@
 	)
 	(segment
-		(start 165.699 99.801)
-		(end 165.75 99.75)
-		(width 0.3)
-		(layer "In1.Cu")
-		(net 33)
-	)
-	(segment
 		(start 166.222 95.422)
 		(end 165.4 94.6)
@@
 	)
 	(segment
-		(start 165.75 99.75)
-		(end 165.75 99.095384)
-		(width 0.3)
-		(layer "In1.Cu")
-		(net 33)
-	)
-	(segment
 		(start 165.4 94.6)
 		(end 164.820768 94.6)
@@
 	)
 	(segment
-		(start 164.551 99.801)
-		(end 165.699 99.801)
-		(width 0.3)
-		(layer "In1.Cu")
-		(net 33)
-	)
-	(segment
-		(start 163.25 98.5)
-		(end 164.551 99.801)
+		(start 165.75 99.65)
+		(end 165.4 100)
 		(width 0.3)
 		(layer "In1.Cu")
@@
 	)
 	(segment
+		(start 165.75 99.095384)
+		(end 165.75 99.65)
+		(width 0.3)
+		(layer "In1.Cu")
+		(net 33)
+	)
+	(segment
 		(start 163.1 96.9)
 		(end 163 97)
@@
 	)
 	(segment
-		(start 165.1 100.9)
-		(end 165.5 100.5)
+		(start 164.1375 100.9)
+		(end 165.3 100.9)
 		(width 0.2)
 		(layer "F.Cu")
@@
 	)
 	(segment
-		(start 164.1375 100.9)
-		(end 165.1 100.9)
+		(start 165.3 100.9)
+		(end 165.6 100.6)
 		(width 0.2)
 		(layer "F.Cu")
@@
 	)
 	(via
-		(at 165.5 100.5)
+		(at 165.6 100.6)
 		(size 0.45)
 		(drill 0.3)
@@
 		(width 0.3)
 		(layer "In1.Cu")
-		(net 37)
-	)
-	(segment
-		(start 165.6 100.6)
-		(end 165.5 100.5)
-		(width 0.3)
-		(layer "In1.Cu")

Commit message: Various stuff
Parts:
- C20: value 0.1uF -> 100nF
Routing:
- net GPIO16: track 32.6 -> 28.9 mm
- net +3V3: track 97.7 -> 96.5 mm
- net SWCLK: track 33.6 -> 33.5 mm, vias 4 -> 2

Commit message: Cleanup, documentation
Parts:
- J1: footprint Connector_USB:USB_C_Receptacle_HRO_TYPE-C-31-M-12 -> pico-2v:USB_C_Receptacle_HRO_TYPE-C-31-M-12
- SW1: value UK-B0273-SP25Y -> KMR231GLFS
- SW2: value USB Boot -> KMR231GLFS
