File: pico-2v.kicad_sch (KiCad schematic)
At the start: 49 parts, among them J1 USB_C_Receptacle_USB2.0_16P, J2 VOLTSEL, J3 Header-1, J4 Header-2, J5 Conn_01x04, J6 Conn_01x04, J7 Conn_02x05_Odd_Even, SW1 UK-B0273-SP25Y, SW2 USB Boot, U1 RP2354A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

Commit message: Stuff
Parts:
- added D2: RED, LED_SMD:LED_0603_1608Metric, symbol Device:LED
- added R12: 470R, Resistor_SMD:R_0402_1005Metric, symbol Device:R
Connections:
- net GND: now also R12.1
- net USB_D+: no longer R3.1, U1.52 (USB_DP)
- net USB_D-: no longer R4.2, U1.51 (USB_DM)
- net GPIO25: now reaches U1.37 (GPIO25)
- net GPIO25: now also D2.2 (A)
- new net: D2.1 (K), R12.2
- new net USB_DM: R4.2, U1.51 (USB_DM)
- new net USB_DP: R3.1, U1.52 (USB_DP)
- no-connect marks 13 -> 12
Other:
- note added: "USER LED"
- moved on the sheet: D3, J7, R5

Commit message: Various stuff
Parts:
- C20: value 0.1uF -> 100nF
- SW2: value USB Boot -> UK-B0273-SP25Y; Name (none) -> USB Boot
Changed lines of the file:
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@@
 		(on_board yes)
 		(dnp no)
-		(fields_autoplaced yes)
 		(property "Reference" "SW2"
 			(at 201.93 83.8199 90)
@@
 				)
 				(justify right)
-				(hide yes)
 			)
 		)
-		(property "Value" "USB Boot"
+		(property "Value" "UK-B0273-SP25Y"
 			(at 201.93 86.3599 90)
 			(effects
@@
 			)
 		)
+		(property "Name" "USB Boot"
+			(at 206.502 88.392 90)
+			(effects
+				(font
+					(size 1.27 1.27)
+				)
+			)
+		)
 		(pin "2"
 		)
@@
 			)
 		)
-		(property "Value" "0.1uF"
+		(property "Value" "100nF"
 			(at 283.464 80.01 0)
 			(effects

Commit message: Cleanup, documentation
Parts:
- J1: footprint Connector_USB:USB_C_Receptacle_HRO_TYPE-C-31-M-12 -> pico-2v:USB_C_Receptacle_HRO_TYPE-C-31-M-12
- SW1, SW2: value UK-B0273-SP25Y -> KMR231GLFS
Changed lines of the file:
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@@
 			)
 		)
-		(property "Value" "UK-B0273-SP25Y"
+		(property "Value" "KMR231GLFS"
 			(at 201.93 86.3599 90)
 			(effects
@@
 			)
 		)
-		(property "Value" "UK-B0273-SP25Y"
+		(property "Value" "KMR231GLFS"
 			(at 256.54 78.232 0)
 			(effects
@@
 			)
 		)
-		(property "Footprint" "Connector_USB:USB_C_Receptacle_HRO_TYPE-C-31-M-12"
+		(property "Footprint" "pico-2v:USB_C_Receptacle_HRO_TYPE-C-31-M-12"
 			(at 358.14 58.42 0)
 			(effects
